File: vfc_power_supply.kicad_pcb (KiCad board)
At the start: 2 copper layers, 65 x 56 mm, 5 parts, among them P1 Conn_02x20_Odd_Even

Commit message: more progress
Parts:
- added C1: 10u, Capacitor_SMD:C_1210_3225Metric, F.Cu at (240.8, 125.0)
- added C10: 100n, Capacitor_SMD:C_0402_1005Metric, F.Cu at (230.5, 112.0)
- added C11: 10u, Capacitor_SMD:C_1210_3225Metric, F.Cu at (252.8, 116.0)
- added C12: 10u, Capacitor_SMD:C_1210_3225Metric, F.Cu at (242.0, 116.1)
- added C14: 1u, Capacitor_SMD:C_0402_1005Metric, F.Cu at (233.2, 111.8)
- added C15: 1u, Capacitor_SMD:C_0402_1005Metric, F.Cu at (233.2, 117.2)
- added C16: 12p, Capacitor_SMD:C_0402_1005Metric, F.Cu at (238.5, 113.0)
- added C17: 100u, Capacitor_WUT:Wurth_WCAP_PSHP, F.Cu at (228.8, 105.5)
- added C18: 1u, Capacitor_SMD:C_0402_1005Metric, F.Cu at (236.0, 110.8)
- added C19: 100n, Capacitor_SMD:C_0402_1005Metric, F.Cu at (239.0, 114.5)
- added C2: 1u, Capacitor_SMD:C_0402_1005Metric, F.Cu at (245.2, 125.2)
- added C20: 100n, Capacitor_SMD:C_0402_1005Metric, F.Cu at (219.0, 111.2)
- added C4: 4p7, Capacitor_SMD:C_0402_1005Metric, F.Cu at (249.2, 130.0)
- added C5: 100u, Capacitor_WUT:Wurth_WCAP_PSHP, F.Cu at (233.0, 134.5)
- added C6: 10n, Capacitor_SMD:C_0402_1005Metric, B.Cu at (248.8, 129.5)
- added C7: 10n, Capacitor_SMD:C_0402_1005Metric, B.Cu at (248.8, 128.5)
- added C8: 4p7, Capacitor_SMD:C_0402_1005Metric, F.Cu at (248.2, 127.5)
- added C9: 100u, Capacitor_WUT:Wurth_WCAP_PSHP, F.Cu at (256.0, 131.5)
- added J1: Connector_RJ45_Magjack_Abracon_ARJM11D7-502-AB-EW2, Connector_WUT:Connector_RJ45_Magjack_Abracon_ARJM11D7-502-AB-EW2, F.Cu at (206.0, 111.8)
- added J2: Connector_RJ45_Magjack_Abracon_ARJ146, Connector_WUT:Connector_RJ45_Magjack_Abracon_ARJ146, F.Cu at (202.8, 132.0)
- added J3: Conn_01x03_Male, Connector_WUT:Powerpole_PP30-with-1377G2-PCB-pins-25A_3WAY, B.Cu at (249.0, 122.5)
- added L1: 12u, Inductor_SMD:L_Coilcraft_LPS5030, F.Cu at (241.2, 134.8)
- added L2: 6u8, Inductor_SMD:L_Coilcraft_LPS4018, F.Cu at (248.0, 135.0)
- added L3: 74279226101, Inductor_SMD:L_1812_4532Metric, F.Cu at (247.0, 117.5)
- added L4: 1u5, Inductor_SMD:L_Coilcraft_XAL60xx_6.36x6.56mm, F.Cu at (226.5, 114.2)
- added R1: 270k, Resistor_SMD:R_0402_1005Metric, F.Cu at (242.2, 127.8)
- added R10: 4k7, Resistor_SMD:R_0402_1005Metric, F.Cu at (235.5, 118.5)
- added R11: 18k, Resistor_SMD:R_0402_1005Metric, F.Cu at (237.5, 115.8)
- added R12: 240k, Resistor_SMD:R_0402_1005Metric, F.Cu at (239.5, 113.0)
- added R13: DNF, Resistor_SMD:R_0805_2012Metric, B.Cu at (209.8, 144.5)
- added R2: DNF, Resistor_SMD:R_0402_1005Metric, F.Cu at (241.0, 127.8)
- added R3: 1M, Resistor_SMD:R_0402_1005Metric, F.Cu at (248.2, 130.0)
- added R4: 39k, Resistor_SMD:R_0402_1005Metric, F.Cu at (250.2, 130.0)
- added R5: 15k, Resistor_SMD:R_0402_1005Metric, F.Cu at (246.8, 125.8)
- added R6: 1M, Resistor_SMD:R_0402_1005Metric, F.Cu at (249.2, 127.5)
- added R7: 71k5, Resistor_SMD:R_0402_1005Metric, F.Cu at (250.2, 127.5)
- added R8: 91k, Resistor_SMD:R_0402_1005Metric, F.Cu at (233.2, 118.5)
- added R9: 1M, Resistor_SMD:R_0402_1005Metric, F.Cu at (237.5, 113.0)
- added TP1: ~, TestPoint:TestPoint_THTPad_D2.0mm_Drill1.0mm, F.Cu at (236.5, 143.2)
- added TP2: ~, TestPoint:TestPoint_THTPad_D2.0mm_Drill1.0mm, F.Cu at (256.2, 140.8)
- added TP3: ~, TestPoint:TestPoint_THTPad_D2.0mm_Drill1.0mm, F.Cu at (220.0, 102.8)
- added U1: LT8653S, IC_WUT:LQFN-20-1EP_3x4mm_P0.5mm_EP1.4x2.4mm, F.Cu at (245.0, 129.0)
- added U2: LT8636, IC_WUT:LQFN-20-1EP_3x4mm_P0.5mm_EP1.65x2.65mm, F.Cu at (234.2, 114.2)
- added U3: LTC2497, IC_WUT:QFN-38-1EP_5x7mm_P0.5mm_EP3.15x5.15mm, F.Cu at (251.0, 106.5)
- MK1, MK4: footprint MountingHole:MountingHole_2.7mm_M2.5 -> MountingHole:MountingHole_2.7mm_M2.5_Pad_Via
- MK2: renamed from MK3; footprint MountingHole:MountingHole_2.7mm_M2.5 -> MountingHole:MountingHole_2.7mm_M2.5_Pad_Via
- MK3: renamed from MK2; footprint MountingHole:MountingHole_2.7mm_M2.5 -> MountingHole:MountingHole_2.7mm_Pad_Via
Connections:
- P1 pad 17: +3V3 -> Net-(P1-Pad17)
Routing:
- net /PoE Injector/D4_P: track 0.00 -> 48.0 mm
- net /PoE Injector/D4_N: track 0.00 -> 46.6 mm
- net /PoE Injector/D2_P: track 0.00 -> 45.0 mm
- net /PoE Injector/D3_P: track 0.00 -> 45.0 mm
- net /PoE Injector/D1_P: track 0.00 -> 45.0 mm
- net /PoE Injector/D3_N: track 0.00 -> 45.0 mm
- net /PoE Injector/D1_N: track 0.00 -> 44.8 mm
- net /PoE Injector/D2_N: track 0.00 -> 44.3 mm
- net +12V: track 0.00 -> 26.3 mm
- net /Power Supplies/PG_5V: track 0.00 -> 24.9 mm, vias 0 -> 3
- net +5V: track 0.00 -> 24.6 mm, vias 0 -> 6
- net GND: track 0.00 -> 22.6 mm, vias 0 -> 56
- net Net-(U1-Pad6): track 0.00 -> 21.1 mm, vias 0 -> 2
- net Net-(C1-Pad1): track 0.00 -> 12.1 mm, vias 0 -> 4
- net VCC: track 0.00 -> 9.47 mm, vias 0 -> 3
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- added copper zone on F.Cu, net +12V
- added copper zone on F.Cu, net +5V
- added copper zone on In2.Cu, net +5V
- added copper zone on F.Cu, net /VIN
- added copper zone on F.Cu, net GND
- added copper zone on In1.Cu, net GND
- added copper zone on B.Cu, net GNDA
- added copper zone on F.Cu, net Net-(C1-Pad1)
- added copper zone on In2.Cu, net Net-(C1-Pad1)
- added copper zone on F.Cu, net Net-(C10-Pad2)
- added copper zone on F.Cu, net Net-(L1-Pad1)
- added copper zone on F.Cu, net Net-(L2-Pad1)
- added copper zone on F.Cu, net VDD
- added copper zone on In2.Cu, net VDD
Other:
- outline, holes or cut-outs redrawn
- copper layers 2 -> 4
- net class Default: clearance 0.2 -> 0.16
- net class Ethernet added: clearance 0.16, trace_width 0.25, via_dia 0.9, via_drill 0.6
- rule trace_clearance: 0.2 -> 0.16
- rule via_min_drill: 0.5 -> 0.2
- rule via_min_size: 0.8 -> 0.4
- board text removed: "CAMERA"
- board text removed: "DISPLAY"
