File: vfc_power_supply.kicad_pcb (KiCad board)
At the start: 4 copper layers, 65 x 56 mm, 74 parts, among them J1 Connector_RJ45_Magjack_Abraco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, J2 Connector_RJ45_Magjack_Abraco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, J3 Conn_01x03_Male, J4 Conn_02x08_Odd_Even, M1 Logo_10mmx10mm, P1 Conn_02x20_Odd_Even, U1 LT8653S, U2 LT8636, U3 LTC2497, U4 REF5030ID, U5 PCT2075D

Commit message: Ready for review
Parts:
- removed the J4 at (260.5, 102.0)
- removed the R29 at (257.5, 114.5)
- added C25: 1u, Capacitor_SMD:C_0402_1005Metric, F.Cu at (254.2, 118.3)
- added C26: 1u, Capacitor_SMD:C_0402_1005Metric, F.Cu at (244.5, 118.3)
- added D1: 3V3, Diode_SMD:D_SOD-523, B.Cu at (250.5, 102.0)
- added D10: 3V3, Diode_SMD:D_SOD-523, B.Cu at (252.2, 114.5)
- added D11: 3V3, Diode_SMD:D_SOD-523, B.Cu at (250.8, 114.5)
- added D12: 3V3, Diode_SMD:D_SOD-523, B.Cu at (249.2, 114.5)
- added D2: 3V3, Diode_SMD:D_SOD-523, B.Cu at (254.8, 111.8)
- added D3: 3V3, Diode_SMD:D_SOD-523, B.Cu at (252.0, 102.0)
- added D4: 3V3, Diode_SMD:D_SOD-523, F.Cu at (258.0, 107.2)
- added D5: 3V3, Diode_SMD:D_SOD-523, B.Cu at (253.5, 102.0)
- added D6: 3V3, Diode_SMD:D_SOD-523, B.Cu at (255.0, 102.0)
- added D7: 3V3, Diode_SMD:D_SOD-523, B.Cu at (256.5, 102.0)
- added D8: 3V3, Diode_SMD:D_SOD-523, B.Cu at (258.0, 102.0)
- added D9: 3V3, Diode_SMD:D_SOD-523, B.Cu at (253.8, 114.5)
- added J1: Conn_02x08_Odd_Even, Connector_PinHeader_2.54mm:PinHeader_2x08_P2.54mm_Vertical, F.Cu at (260.5, 102.0)
- added J5: Connector_RJ45_Magjack_Abracon_ARJ146, Connector_WUT:Connector_RJ45_Magjack_Abracon_ARJ146, F.Cu at (254.8, 147.2)
- added R1: R, Resistor_SMD:R_0402_1005Metric, F.Cu at (234.8, 114.2)
- added R12: R, Resistor_SMD:R_0402_1005Metric, B.Cu at (257.5, 114.5)
- added R13: 390k, Resistor_SMD:R_0402_1005Metric, F.Cu at (238.5, 120.0)
- added R14: 560k, Resistor_SMD:R_0402_1005Metric, F.Cu at (248.2, 120.0)
- added R2: R, Resistor_SMD:R_0402_1005Metric, F.Cu at (247.2, 114.8)
- added R3: R, Resistor_SMD:R_0402_1005Metric, F.Cu at (236.8, 106.0)
- added R36: 10K, Resistor_SMD:R_0402_1005Metric, F.Cu at (254.2, 120.2)
- added R37: 10K, Resistor_SMD:R_0402_1005Metric, F.Cu at (248.2, 119.0)
- added R38: 10K, Resistor_SMD:R_0402_1005Metric, F.Cu at (246.2, 120.8)
- added R39: 10K, Resistor_SMD:R_0402_1005Metric, F.Cu at (244.5, 120.2)
- added R4: R, Resistor_SMD:R_0402_1005Metric, F.Cu at (222.0, 117.8)
- added R40: 10K, Resistor_SMD:R_0402_1005Metric, F.Cu at (238.5, 119.0)
- added R41: 10K, Resistor_SMD:R_0402_1005Metric, F.Cu at (238.5, 121.0)
- added U6: FPF2701MPX, IC_WUT:MLP-8-1EP_3x3mm_P0.65mm_EP1.7x2.4mm, F.Cu at (251.5, 119.8)
- added U7: FPF2701MPX, IC_WUT:MLP-8-1EP_3x3mm_P0.65mm_EP1.7x2.4mm, F.Cu at (241.8, 119.8)
- added U8: TVS3300DRV, Package_SON:WSON-6-1EP_2x2mm_P0.65mm_EP1x1.6mm, B.Cu at (261.8, 133.0)
- J2: value Connector_RJ45_Magjack_Abracon_ARJ146 -> Conn_01x02_Male; footprint Connector_WUT:Connector_RJ45_Magjack_Abracon_ARJ146 -> Connector_Molex:Molex_KK-254_AE-6410-02A_1x02_P2.54mm_Vertical
- moved M1 54.0 mm to (191.0, 106.8)
- moved J2 29.0 mm to (238.5, 123.2), turned to 270 degrees
- moved TP3 18.3 mm to (217.0, 105.8)
- moved C11 7.70 mm to (209.0, 124.0), turned to 270 degrees
- moved TP1 6.56 mm to (233.0, 112.2)
- moved LD1 3.02 mm to (212.2, 102.5)
- moved R15 3.02 mm to (216.5, 101.2)
- moved R16 3.02 mm to (216.5, 102.5)
- moved R17 3.02 mm to (216.5, 103.8)
- moved C12 2.30 mm to (213.4, 117.5)
- moved R27 1.80 mm to (213.5, 114.2), turned to 90 degrees
- moved C1 1.50 mm to (219.2, 116.8)
- moved C2 1.50 mm to (219.5, 112.2)
- moved C3 1.50 mm to (224.2, 108.2)
- moved C4 1.50 mm to (228.8, 124.5)
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- renumbered C14 to C13, C15 to C14, C16 to C15, C17 to C16, C23 to C17, C24 to C20, C13 to C21, C21 to C22, C3 to C23, C20 to C24, C4 to C3, C5 to C4, C6 to C5, C7 to C6, C8 to C7, C9 to C8, C22 to C9, J1 to J4, R27 to R10, R28 to R11, R17 to R15, R18 to R16, R19 to R17, R20 to R18, R21 to R19, R1 to R20, R2 to R21, R3 to R22, R4 to R23, R5 to R24, R6 to R25, R7 to R26, R8 to R27, R9 to R28, R10 to R29, R11 to R30, R12 to R31, R16 to R32, R14 to R33, R15 to R34, R13 to R35, R22 to R5, R23 to R6, R24 to R7, R25 to R8, R26 to R9, U4 to U3, U5 to U4, U3 to U5
Connections:
- net /GPIO10(SPI0_MOSI) renamed Net-(P1-Pad19)
- net /GPIO12(PWM0) renamed Net-(P1-Pad32)
- net /GPIO14(TXD0) renamed Net-(P1-Pad8)
- net /GPIO15(RXD0) renamed Net-(P1-Pad10)
- net /GPIO16 renamed Net-(P1-Pad36)
- net /GPIO17(GEN0) renamed /RGB_BLUE
- net /GPIO18(GEN1)(PWM0) renamed Net-(P1-Pad12)
- net /GPIO2(SDA1) renamed /SDA
- net /GPIO20(SPI1_MOSI) renamed Net-(P1-Pad38)
- net /GPIO21(SPI1_SCK) renamed Net-(P1-Pad40)
- net /GPIO22(GEN3) renamed /RGB_RED
- net /GPIO23(GEN4) renamed /PGOOD_12V
- net /GPIO24(GEN5) renamed /PGOOD_21V
- net /GPIO25(GEN6) renamed Net-(P1-Pad22)
- net /GPIO26 renamed Net-(P1-Pad37)
- net /GPIO27(GEN2) renamed /RGB_GREEN
- net /GPIO3(SCL1) renamed /SCL
- net /GPIO4(GCLK) renamed Net-(P1-Pad7)
- net /GPIO8(SPI0_CE_N) renamed Net-(P1-Pad24)
- net /GPIO9(SPI0_MISO) renamed Net-(P1-Pad21)
- net /ID_SC renamed Net-(P1-Pad28)
- net /ID_SD renamed Net-(P1-Pad27)
- net Net-(C1-Pad1) renamed /VIN_CLEAN
- J2 pad 1: Net-(J2-Pad1) -> /Network Switch Load Switch/VOUT
- J2 pad 2: /PoE Injector/D3_N -> GND
- P1 pad 23: /GPIO11(SPI0_SCK) -> /PGOOD_SWITCH
- P1 pad 26: /GPIO7(SPI1_CE_N) -> /~EN_SWITCH
- P1 pad 29: /GPIO5 -> /~FAULT_SWITCH
- P1 pad 31: /GPIO6 -> /PGOOD_POE
- P1 pad 33: /GPIO13(PWM1) -> /~EN_POE
- P1 pad 35: /GPIO19(SPI1_MISO) -> /~FAULT_POE
- RN2 pad 1: /ADC/CH7 -> Net-(RN2-Pad1)
- RN2 pad 2: /ADC/CH6 -> Net-(RN2-Pad2)
- RN2 pad 3: /ADC/CH5 -> Net-(RN2-Pad3)
- RN2 pad 4: /ADC/CH4 -> Net-(RN2-Pad4)
- U5 pad 12: /ADC/CH4 -> Net-(U5-Pad12)
- U5 pad 13: /ADC/CH5 -> Net-(U5-Pad13)
- U5 pad 14: /ADC/CH6 -> Net-(U5-Pad14)
- U5 pad 15: /ADC/CH7 -> Net-(U5-Pad15)
Routing:
- net /ADC/CH3: track 3.11 -> 43.2 mm, vias 0 -> 4
- net /~EN_POE: track 0.00 -> 33.8 mm, vias 0 -> 1
- net +3V3: track 39.2 -> 72.5 mm, vias 2 -> 7
- net /PoE Injector/VDD_AP: track 0.00 -> 28.5 mm, vias 0 -> 1
- net /~EN_SWITCH: track 0.00 -> 28.4 mm, vias 0 -> 3
- net /~FAULT_POE: track 0.00 -> 27.9 mm, vias 0 -> 1
- net /~FAULT_SWITCH: track 0.00 -> 25.8 mm, vias 0 -> 2
- net /Network Switch Load Switch/VOUT: track 0.00 -> 25.1 mm
- net /PGOOD_SWITCH: track 0.00 -> 23.3 mm, vias 0 -> 3
- net /PGOOD_POE: track 0.00 -> 23.1 mm, vias 0 -> 1
- net /ADC/CH2: track 3.23 -> 23.8 mm, vias 0 -> 2
- net /ADC/CH0: track 3.92 -> 22.0 mm, vias 0 -> 2
- net /ADC/CH1: track 3.51 -> 11.5 mm, vias 0 -> 1
- net +12V: track 17.5 -> 24.5 mm, vias 0 -> 7
- net /ADC/CH7: track 6.48 -> 0.00 mm
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- added copper zone on In2.Cu, net +12V
- added copper zone on In2.Cu, net GND
Other:
- board text added: "0V"
- board text added: "11"
- board text added: "12V"
- board text added: "24V"
- board text added: "5V"
- board text added: "8"
- board text added: "CH12"
- board text added: "CH14"
- board text added: "CH15"
- board text added: "CH9"
- board text added: "ETH IN"
- board text added: "ETH+PoE->"
- board text added: "PoE"
- board text removed: "RASPBERRY-PI 40-PIN ADDON BOARD VIEW FROM TOP NOTE: P1 SHOULD BE FITTED ON THE REVERSE OF THE BOARD ADD EDGE CUTS FROM CAMERA AND DISPLAY PORTS AS REQUIRED"

Commit message: Commit before restarting layout
Parts:
- L1: footprint Inductor_SMD:L_Coilcraft_LPS5030 -> Inductor_WUT:Coilcraft_LPS5030
- L2: footprint Inductor_SMD:L_Coilcraft_LPS4018 -> Inductor_WUT:Coilcraft_LPS4018
- L4: footprint Inductor_SMD:L_Coilcraft_XAL60xx_6.36x6.56mm -> Inductor_WUT:Coilcraft_XEL6030
- LD1: footprint LED_SMD:LED_RGB_PLCC-6 -> LED_WUT:LED_Cree_CLX6E-FKC
- R1, R4: value R -> 100k
- R2: value R -> 47k
- R3: value R -> 10k
- U4: footprint Package_SO:SO-8_3.9x4.9mm_P1.27mm -> Package_SO:SOIC-8_3.9x4.9mm_P1.27mm
- U6, U7: footprint IC_WUT:MLP-8-1EP_3x3mm_P0.65mm_EP1.7x2.4mm -> IC_WUT:WDFN-8-1EP_3x3mm_P0.65mm_EP1.7x2.52mm
- moved M1 30.7 mm to (214.2, 126.8)
- moved R41 6.01 mm to (238.2, 115.0), turned to -90 degrees
- moved R39 5.73 mm to (238.8, 121.0), turned to 0 degrees
- moved R13 5.06 mm to (239.2, 115.0), turned to 90 degrees
- moved C26 4.60 mm to (240.8, 121.0), turned to 0 degrees
- moved R40 4.37 mm to (240.2, 115.0), turned to -90 degrees
- moved U7 2.86 mm to (239.3, 118.2), turned to -90 degrees
- moved R1 1.25 mm to (235.5, 113.2)
- moved C11 1.03 mm to (208.0, 124.2)
Connections:
- net /ADC/CH0 renamed /CH0
- net /ADC/CH1 renamed /CH1
- net /ADC/CH10 renamed /CH10
- net /ADC/CH11 renamed /CH11
- net /ADC/CH12 renamed /CH12
- net /ADC/CH13 renamed /CH13
- net /ADC/CH14 renamed /CH14
- net /ADC/CH15 renamed /CH15
- net /ADC/CH2 renamed /CH2
- net /ADC/CH3 renamed /CH3
- net /ADC/CH8 renamed /CH8
- net /ADC/CH9 renamed /CH9
- net /Network Switch Load Switch/ISET renamed /ISET_1
- net /Network Switch Load Switch/VOUT renamed /VOUT
- net /PoE Injector/VDD_AP renamed /VOUT_1
- net /PoE Load Switch/ISET renamed /ISET
- net Net-(J4-PadL1) renamed no_connect_80
- net Net-(J4-PadL2) renamed no_connect_81
- net Net-(J4-PadL3) renamed no_connect_82
- net Net-(J4-PadL4) renamed no_connect_83
- net Net-(J5-Pad1) renamed no_connect_84
- net Net-(J5-Pad12) renamed no_connect_85
- net Net-(J5-Pad13) renamed no_connect_86
- net Net-(J5-Pad14) renamed no_connect_87
- net Net-(J5-Pad6) renamed no_connect_88
- net Net-(J5-Pad7) renamed no_connect_89
- net Net-(P1-Pad1) renamed no_connect_90
- net Net-(P1-Pad10) renamed no_connect_91
- net Net-(P1-Pad12) renamed no_connect_92
- net Net-(P1-Pad19) renamed no_connect_93
- net Net-(P1-Pad21) renamed no_connect_94
- net Net-(P1-Pad22) renamed no_connect_95
- net Net-(P1-Pad24) renamed no_connect_96
- net Net-(P1-Pad27) renamed no_connect_97
- net Net-(P1-Pad28) renamed no_connect_98
- net Net-(P1-Pad32) renamed no_connect_99
- net Net-(P1-Pad36) renamed no_connect_100
- net Net-(P1-Pad37) renamed no_connect_101
- net Net-(P1-Pad38) renamed no_connect_102
- net Net-(P1-Pad40) renamed no_connect_103
- net Net-(P1-Pad7) renamed no_connect_104
- net Net-(P1-Pad8) renamed no_connect_105
- net Net-(RN2-Pad1) renamed no_connect_106
- net Net-(RN2-Pad2) renamed no_connect_107
- net Net-(RN2-Pad3) renamed no_connect_108
- net Net-(RN2-Pad4) renamed no_connect_109
- net Net-(U2-Pad16) renamed no_connect_110
- net Net-(U3-Pad3) renamed no_connect_111
- net Net-(U3-Pad5) renamed no_connect_112
- net Net-(U4-Pad3) renamed no_connect_113
- net Net-(U5-Pad12) renamed no_connect_114
- net Net-(U5-Pad13) renamed no_connect_115
- net Net-(U5-Pad14) renamed no_connect_116
- net Net-(U5-Pad15) renamed no_connect_117
- U3 pad 1: Net-(U3-Pad1) -> (no net)
- U3 pad 7: Net-(U3-Pad7) -> (no net)
- U3 pad 8: Net-(U3-Pad8) -> (no net)
Routing:
- net /VOUT: track 25.1 -> 6.31 mm
- net +3V3: track 72.5 -> 81.7 mm, vias 7 -> 8
- net VDDA: track 28.4 -> 37.4 mm
- net /~EN_SWITCH: track 28.4 -> 24.9 mm, vias 3 -> 2
- net /~FAULT_SWITCH: track 25.8 -> 29.0 mm, vias 2 -> 3
- net /CH3: track 43.2 -> 41.0 mm, vias 4 -> 2
- net /PoE Injector/D4_N: track 46.6 -> 48.3 mm
- net GND: track 72.8 -> 71.3 mm, vias 128 -> 123
- net /PGOOD_SWITCH: track 23.3 -> 24.2 mm
- net /PoE Injector/D4_P: track 48.0 -> 47.5 mm
- net +12V: track 24.5 -> 24.0 mm, vias 7 -> 5
Other:
- net class Default removed
- net class Ethernet removed
- net class Power removed
- board text added: "PoE->"
- board text removed: "ETH+PoE->"

Commit message: Updated library parts
Parts:
- removed P1: Conn_02x20_Odd_Even, Connector_PinSocket_2.54mm:PinSocket_2x20_P2.54mm_Vertical
- added J6: Raspberry_Pi_4B, Modules_WUT:Raspberry_Pi_4B, F.Cu at (93.0, 80.0)
- C5, C6, D1, D10, D11, D12, D2, D3, D5, D6, D7, D8, D9, R10, R11, R12, R35, R5, R6, R7, R8, R9, U8: moved to F.Cu
- moved R37 209.9 mm to (441.4, 36.7)
- moved R38 205.4 mm to (436.5, 43.3)
- moved U6 203.3 mm to (437.6, 38.0)
- moved C25 200.5 mm to (439.4, 41.3), turned to 0 degrees
- moved R36 198.6 mm to (436.5, 41.3), turned to 0 degrees
- moved R35 176.7 mm to (388.8, 71.3), turned to 0 degrees
- moved M1 169.8 mm to (360.9, 41.2)
- moved C24 169.5 mm to (392.4, 70.8), turned to 0 degrees
- moved LD1 169.4 mm to (369.0, 38.2)
- moved C21 167.2 mm to (403.9, 98.9), turned to 0 degrees
- moved R33 165.3 mm to (410.4, 91.6), turned to 0 degrees
- moved R32 164.8 mm to (410.4, 93.6), turned to 0 degrees
- moved C20 163.6 mm to (400.3, 102.9), turned to 0 degrees
- moved U8 163.2 mm to (408.3, 61.1)
- moved D12 159.2 mm to (407.2, 94.2), turned to 0 degrees
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Routing:
- net +3V3: track 81.7 -> 0.00 mm, vias 8 -> 0
- net GND: track 71.3 -> 0.00 mm, vias 123 -> 0
- net /SDA: track 52.3 -> 0.00 mm, vias 1 -> 0
- net /SCL: track 48.4 -> 0.00 mm, vias 1 -> 0
- net /PoE Injector/D4_N: track 48.3 -> 0.00 mm
- net /PoE Injector/D4_P: track 47.5 -> 0.00 mm
- net /PoE Injector/D2_P: track 45.0 -> 0.00 mm
- net /PoE Injector/D3_P: track 45.0 -> 0.00 mm
- net /PoE Injector/D1_P: track 45.0 -> 0.00 mm
- net /PoE Injector/D3_N: track 45.0 -> 0.00 mm
- net /PoE Injector/D1_N: track 44.8 -> 0.00 mm
- net /PoE Injector/D2_N: track 44.3 -> 0.00 mm
- net /CH3: track 41.0 -> 0.00 mm, vias 2 -> 0
- net VDDA: track 37.4 -> 0.00 mm
- net /~EN_POE: track 33.8 -> 0.00 mm, vias 1 -> 0
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- removed copper zone on F.Cu, net +12V
- removed copper zone on In2.Cu, net +12V
- removed copper zone on F.Cu, net +5V
- removed copper zone on In2.Cu, net +5V
- removed copper zone on F.Cu, net /VIN
- removed copper zone on F.Cu, net /VIN_CLEAN
- removed copper zone on In2.Cu, net /VIN_CLEAN
- removed copper zone on B.Cu, net GND
- removed copper zone on F.Cu, net GND
- removed copper zone on In1.Cu, net GND
- removed copper zone on In2.Cu, net GND
- removed copper zone on B.Cu, net GNDA
- removed copper zone on F.Cu, net Net-(C10-Pad2)
- removed copper zone on F.Cu, net Net-(L1-Pad1)
- removed copper zone on F.Cu, net Net-(L2-Pad1)
- removed copper zone on F.Cu, net VDD
- removed copper zone on In2.Cu, net VDD
Other:
- board size 65 x 56 mm -> 89.2 x 124.8 mm
- copper layers 4 -> 2
- board text removed: "0V"
- board text removed: "11"
- board text removed: "12V"
- board text removed: "24V"
- board text removed: "5V"
- board text removed: "8"
- board text removed: "CH12"
- board text removed: "CH14"
- board text removed: "CH15"
- board text removed: "CH9"
- board text removed: "ETH IN"
- board text removed: "PoE"
- board text removed: "PoE->"
- board text removed: "RJ45"
- board text removed: "USB"

Commit message: new layout
Parts:
- moved C23 499.0 mm to (-53.5, 287.7)
- moved C25 499.0 mm to (-21.5, 232.5)
- moved D5 499.0 mm to (-60.2, 289.4)
- moved D8 499.0 mm to (-60.2, 291.9)
- moved J1 499.0 mm to (-109.7, 229.2)
- moved J2 499.0 mm to (-142.7, 283.7)
- moved R13 499.0 mm to (-110.5, 250.3)
- moved R17 499.0 mm to (-130.6, 267.0)
- moved R24 499.0 mm to (-125.6, 309.8)
- moved R26 499.0 mm to (-135.6, 309.7)
- moved R31 499.0 mm to (-125.6, 307.8)
- moved R9 499.0 mm to (-130.6, 265.0)
- moved RN2 499.0 mm to (-63.9, 292.2)
- moved TP2 499.0 mm to (-117.1, 297.5)
- moved U5 499.0 mm to (-70.7, 286.0)
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Connections:
- C25 pad 1: /VOUT_1 -> /VOUT
- C26 pad 1: /VOUT -> /VOUT_1
- J2 pad 1: /VOUT -> /VOUT_1
- J5 pad 15: /VOUT_1 -> /VOUT
- U6 pad 8: /VOUT_1 -> /VOUT
- U7 pad 8: /VOUT -> /VOUT_1
- U8 pad 4: /VOUT_1 -> /VOUT
- U8 pad 5: /VOUT_1 -> /VOUT
- U8 pad 6: /VOUT_1 -> /VOUT
Other:
- board size 89.2 x 124.8 mm -> 100 x 130 mm

Commit message: Started new connector layout
Parts:
- removed D10, D11, D12, D6, D7, D8, D9: 3V3, Diode_SMD:D_SOD-523
- removed RN2: 10k, Resistor_SMD:R_Cat16-8
- added C27: 100n, Capacitor_SMD:C_0402_1005Metric, F.Cu at (-12.0, 93.1)
- added C28: 100n, Capacitor_SMD:C_0402_1005Metric, F.Cu at (-15.6, 95.0)
- added C29: 100n, Capacitor_SMD:C_0402_1005Metric, F.Cu at (-28.7, 111.2)
- added C30: 100n, Capacitor_SMD:C_0402_1005Metric, F.Cu at (-12.7, 95.0)
- added C31: 1u, Capacitor_SMD:C_0402_1005Metric, F.Cu at (-15.6, 97.0)
- added C32: 100n, Capacitor_SMD:C_0402_1005Metric, F.Cu at (-20.9, 101.9)
- added C33: 100n, Capacitor_SMD:C_0402_1005Metric, F.Cu at (-28.4, 147.5)
- added C34: 100n, Capacitor_SMD:C_0402_1005Metric, F.Cu at (-28.7, 109.2)
- added FL1: EMI_Filter_CommonMode, Inductor_WUT:TDK_ACM7060-301-2PL-TL01, F.Cu at (-54.5, 91.2)
- added FL2: EMI_Filter_CommonMode, Inductor_WUT:TDK_ACM7060-301-2PL-TL01, F.Cu at (-76.2, 169.9)
- added LD2: LED_Cree_CLX6E-FKC, LED_WUT:LED_Cree_CLX6E-FKC, F.Cu at (-67.9, 168.8)
- added R42: 10k, Resistor_SMD:R_0402_1005Metric, F.Cu at (-28.6, 107.3)
- added R43: 10k, Resistor_SMD:R_0402_1005Metric, F.Cu at (-18.5, 97.9)
- added U10: LM4040DBZ-3, Package_TO_SOT_SMD:SOT-23, F.Cu at (-27.6, 101.6)
- added U11: PCT2075D, Package_SO:SOIC-8_3.9x4.9mm_P1.27mm, F.Cu at (-27.5, 55.2)
- added U12: ADS7924, Package_DFN_QFN:QFN-16-1EP_3x3mm_P0.5mm_EP1.45x1.45mm_ThermalVias, F.Cu at (-19.0, 90.3)
- added U9: ISO1540, Package_SO:SOIC-8_3.9x4.9mm_P1.27mm, F.Cu at (-25.9, 90.8)
- C1: value 10u -> 47u; footprint Capacitor_SMD:C_1210_3225Metric -> Capacitor_SMD:C_1206_3216Metric
- C10: value 100n -> 47u; footprint Capacitor_SMD:C_0402_1005Metric -> Capacitor_SMD:C_1206_3216Metric
- C11: value 10u -> 100n; footprint Capacitor_SMD:C_1210_3225Metric -> Capacitor_SMD:C_0402_1005Metric
- C13, C2: value 1u -> 10u; footprint Capacitor_SMD:C_0402_1005Metric -> Capacitor_SMD:C_1210_3225Metric
- C15: value 12p -> 1u
- C16: value 47u -> 12p; footprint Capacitor_SMD:C_1206_3216Metric -> Capacitor_SMD:C_0402_1005Metric
- C18: value 1u -> 47u; footprint Capacitor_SMD:C_0402_1005Metric -> Capacitor_SMD:C_1206_3216Metric
- C19, C24: value 100n -> 1u
- C3: value 4p7 -> 1u
- C4: value 100u -> 4p7; footprint Capacitor_WUT:Wurth_WCAP_PSHP -> Capacitor_SMD:C_0402_1005Metric
- C5: value 10n -> 100u; footprint Capacitor_SMD:C_0402_1005Metric -> Capacitor_WUT:Wurth_WCAP_PSHP
- C7: value 4p7 -> 10n
- C8: value 47u -> 4p7; footprint Capacitor_SMD:C_1206_3216Metric -> Capacitor_SMD:C_0402_1005Metric
- J1: value Conn_02x08_Odd_Even -> Conn_01x03_Male; footprint Connector_PinHeader_2.54mm:PinHeader_2x08_P2.54mm_Vertical -> Connector_WUT:Powerpole_PP30-with-1377G2-PCB-pins-25A_3WAY
- J2: value Conn_01x02_Male -> Conn_01x03_Male; footprint Connector_Molex:Molex_KK-254_AE-6410-02A_1x02_P2.54mm_Vertical -> Connector_WUT:Powerpole_PP30-with-1377G2-PCB-pins-25A_3WAY
- J3: value Conn_01x03_Male -> Conn_01x02_Male; footprint Connector_WUT:Powerpole_PP30-with-1377G2-PCB-pins-25A_3WAY -> Connector_WUT:Weidmuller_SL3.5-2-90G
- J4: value Connector_RJ45_Magjack_Abracon_ARJM11D7-502-AB-EW2 -> Raspberry_Pi_4B; footprint Connector_WUT:Connector_RJ45_Magjack_Abracon_ARJM11D7-502-AB-EW2 -> Modules_WUT:Raspberry_Pi_4B
- J5: value Connector_RJ45_Magjack_Abracon_ARJ146 -> Connector_RJ45_Magjack_Abracon_ARJM11D7-502-AB-EW2; footprint Connector_WUT:Connector_RJ45_Magjack_Abracon_ARJ146 -> Connector_WUT:Connector_RJ45_Magjack_Abracon_ARJM11D7-502-AB-EW2
- J6: value Raspberry_Pi_4B -> Connector_RJ45_Magjack_Abracon_ARJ146; footprint Modules_WUT:Raspberry_Pi_4B -> Connector_WUT:Connector_RJ45_Magjack_Abracon_ARJ146
- LD1: value LED_Cree_CLX6E-FKC -> Dialight 553-0112F; footprint LED_WUT:LED_Cree_CLX6E-FKC -> LED_WUT:LED_Dialight_553-0112F
- R10: value R -> 33k
- R11: value R -> 22k
- R12: value R -> 10k
- R13: value 390k -> 10k
- R14: value 560k -> 10k
- R15: value 7k5 -> DNF
- R16: value 33k -> 1M
- R17: value 22k -> 39k
- R18: value 10k -> 15k
- R19: value 10k -> 1M
- R20: value 270k -> 71k5
- R21: value DNF -> 91k
- R23: value 39k -> 4k7
- R24: value 15k -> 18k
- R25: value 1M -> 240k
- R26: value 71k5 -> 10K
- R27: value 91k -> 10K
- R28: value 1M -> 10K
- R29: value 4k7 -> 10K
- R30: value 18k -> 10K
- R31: value 240k -> 10K
- R32: footprint Resistor_SMD:R_0402_1005Metric -> Resistor_SMD:R_0805_2012Metric
- R33: value DNF -> 100
- R34: value DNF -> 100k
- R35: value DNF -> 4k7; footprint Resistor_SMD:R_0805_2012Metric -> Resistor_SMD:R_0402_1005Metric
- R36: value 10K -> 4k7
- R37, R38: value 10K -> 10k
- R39: value 10K -> 100
- R40, R41: value 10K -> DNF
- R5: value R -> 390k
- R6: value R -> 560k
- R7, R8: value R -> 470
- R9: value R -> 7k5
- RN1: footprint Resistor_SMD:R_Cat16-8 -> Resistor_SMD:R_Cat16-4
- U3: value REF5030ID -> FPF2701MPX; footprint Package_SO:SOIC-8_3.9x4.9mm_P1.27mm -> IC_WUT:WDFN-8-1EP_3x3mm_P0.65mm_EP1.7x2.52mm
- U4: value PCT2075D -> FPF2701MPX; footprint Package_SO:SOIC-8_3.9x4.9mm_P1.27mm -> IC_WUT:WDFN-8-1EP_3x3mm_P0.65mm_EP1.7x2.52mm
- U5: value LTC2497 -> TVS3300DRV; footprint IC_WUT:QFN-38-1EP_5x7mm_P0.5mm_EP3.15x5.15mm -> Package_SON:WSON-6-1EP_2x2mm_P0.65mm_EP1x1.6mm
- U6: value FPF2701MPX -> LM3480-3.3; footprint IC_WUT:WDFN-8-1EP_3x3mm_P0.65mm_EP1.7x2.52mm -> Package_TO_SOT_SMD:SOT-23
- U7: value FPF2701MPX -> LM4040DBZ-3; footprint IC_WUT:WDFN-8-1EP_3x3mm_P0.65mm_EP1.7x2.52mm -> Package_TO_SOT_SMD:SOT-23
- U8: value TVS3300DRV -> ADS7924; footprint Package_SON:WSON-6-1EP_2x2mm_P0.65mm_EP1x1.6mm -> Package_DFN_QFN:QFN-16-1EP_3x3mm_P0.5mm_EP1.45x1.45mm_ThermalVias
- moved J1 323.5 mm to (149.0, 35.0), turned to -90 degrees
- moved LD1 317.4 mm to (174.0, 56.0), turned to 90 degrees
- moved J2 315.2 mm to (51.0, 35.0), turned to 90 degrees
- moved U7 223.4 mm to (-13.9, 89.8)
- moved RN1 215.5 mm to (-14.9, 93.1)
- moved R34 211.0 mm to (-18.5, 93.9)
- moved C26 209.2 mm to (-22.2, 104.3)
- moved R39 208.8 mm to (-25.1, 104.8)
- moved R22 199.9 mm to (-58.6, 146.2)
- moved R33 198.3 mm to (-10.0, 88.6)
- moved R7 197.8 mm to (-48.0, 88.6)
- moved U2 195.3 mm to (-62.4, 145.4)
- moved C5 193.7 mm to (-84.3, 144.8)
- moved R1 191.9 mm to (-58.0, 97.7)
- moved R8 191.3 mm to (-55.1, 95.7)
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Connections:
- net no_connect_104 renamed no_connect_(J6-Pad7)
- net no_connect_110 renamed no_connect_(U2-Pad16)
- net no_connect_90 renamed no_connect_(J6-Pad1)
- net no_connect_92 renamed no_connect_(J6-Pad12)
- C1 pad 1: /VIN_CLEAN -> Net-(C1-Pad1)
- C1 pad 2: GND -> Net-(C1-Pad2)
- C10 pad 1: Net-(C10-Pad1) -> +12V
- C10 pad 2: Net-(C10-Pad2) -> GND
- C11 pad 1: /VIN -> Net-(C11-Pad1)
- C11 pad 2: GND -> Net-(C11-Pad2)
- C12 pad 1: /VIN_CLEAN -> /Power Supplies/VIN
- C15 pad 1: +5V -> /VIN_CLEAN
- C15 pad 2: Net-(C15-Pad2) -> GND
- C16 pad 2: GND -> Net-(C16-Pad2)
- C18 pad 1: Net-(C18-Pad1) -> +5V
- C20 pad 1: VDDA -> Net-(C20-Pad1)
- C21 pad 1: +5V -> /Network Switch Load Switch/VOUT
- C22 pad 1: VDDA -> /PoE Injector/VDD_AP
- C23 pad 1: VDDA -> Net-(C23-Pad1)
- C24 pad 1: Net-(C24-Pad1) -> /ADC/VBAT
- C24 pad 2: GND -> GNDD
- C25 pad 1: /VOUT -> Net-(C25-Pad1)
- C25 pad 2: GND -> GNDD
- C26 pad 1: /VOUT_1 -> Net-(C26-Pad1)
- C26 pad 2: GND -> GNDD
- C3 pad 1: VDD -> /VIN_CLEAN
- C3 pad 2: Net-(C3-Pad2) -> GND
- C4 pad 2: GND -> Net-(C4-Pad2)
- C5 pad 1: Net-(C5-Pad1) -> VDD
- C7 pad 1: +12V -> Net-(C7-Pad1)
- C7 pad 2: Net-(C7-Pad2) -> GND
- C8 pad 2: GND -> Net-(C8-Pad2)
- D1 pad 1: /CH15 -> Net-(D1-Pad1)
- D1 pad 2: GND -> GNDD
- D2 pad 1: /CH14 -> /ADC/CH3
- D3 pad 1: /CH13 -> /ADC/CH2
- D4 pad 1: /CH12 -> /ADC/CH1
- D5 pad 1: /CH11 -> /ADC/CH0
- J1 pad 1: Net-(J1-Pad1) -> /Power Supplies/VIN
- J1 pad 2: GND -> no_connect_(J1-Pad2)
- J1 pad 3: Net-(J1-Pad3) -> GND
- J2 pad 1: /VOUT_1 -> Net-(FL1-Pad2)
- J2 pad 2: GND -> no_connect_(J2-Pad2)
- J3 pad 1: /VIN -> Net-(C1-Pad1)
- J3 pad 2: no_connect_79 -> Net-(C1-Pad2)
- J4 pad 1: /PoE Injector/D1_P -> no_connect_(J4-Pad1)
- J4 pad 10: /PoE Injector/D4_N -> no_connect_(J4-Pad10)
- J4 pad 11: GNDA -> /RGB_BLUE
- J4 pad 2: /PoE Injector/D1_N -> +5V
- J4 pad 3: /PoE Injector/D2_P -> /SDA
- J4 pad 4: /PoE Injector/D2_N -> +5V
- J4 pad 5: Net-(C24-Pad1) -> /SCL
- J4 pad 6: Net-(C24-Pad1) -> GND
- J4 pad 7: /PoE Injector/D3_P -> no_connect_(J4-Pad7)
- J4 pad 8: /PoE Injector/D3_N -> /PGOOD_5V
- J4 pad 9: /PoE Injector/D4_P -> GND
- J5 pad 1: no_connect_84 -> /PoE Injector/D1_P
- J5 pad 10: /PoE Injector/D1_N -> /PoE Injector/D4_N
- J5 pad 11: /PoE Injector/D1_P -> GNDA
- J5 pad 2: /PoE Injector/D3_N -> /PoE Injector/D1_N
- J5 pad 3: /PoE Injector/D3_P -> /PoE Injector/D2_P
- J5 pad 4: /PoE Injector/D2_P -> /PoE Injector/D2_N
- J5 pad 5: /PoE Injector/D2_N -> Net-(C23-Pad1)
- J5 pad 6: no_connect_88 -> Net-(C23-Pad1)
- J5 pad 7: no_connect_89 -> /PoE Injector/D3_P
- J5 pad 8: /PoE Injector/D4_P -> /PoE Injector/D3_N
- J5 pad 9: /PoE Injector/D4_N -> /PoE Injector/D4_P
- J6 pad 10: no_connect_91 -> /PoE Injector/D1_N
- J6 pad 11: /RGB_BLUE -> /PoE Injector/D1_P
- J6 pad 13: /RGB_GREEN -> no_connect_(J6-Pad13)
- J6 pad 14: GND -> no_connect_(J6-Pad14)
- J6 pad 15: /RGB_RED -> /PoE Injector/VDD_AP
- J6 pad 16: /PGOOD_12V -> GND
- J6 pad 17: +3V3 -> GNDA
- J6 pad 2: +5V -> /PoE Injector/D3_N
- J6 pad 3: /SDA -> /PoE Injector/D3_P
- J6 pad 4: +5V -> /PoE Injector/D2_P
- J6 pad 5: /SCL -> /PoE Injector/D2_N
- J6 pad 6: GND -> no_connect_(J6-Pad6)
- J6 pad 8: no_connect_105 -> /PoE Injector/D4_P
- J6 pad 9: GND -> /PoE Injector/D4_N
- L3 pad 1: /VIN -> /Power Supplies/VIN
- L4 pad 1: Net-(C10-Pad2) -> Net-(C11-Pad2)
- LD1 pad 2: GND -> Net-(LD1-Pad2)
- R1 pad 2: /CH0 -> /ADC/CH0
- R10 pad 1: Net-(J1-Pad11) -> /RGB_GREEN
- R10 pad 2: /CH13 -> Net-(LD2-Pad5)
- R11 pad 1: Net-(J1-Pad13) -> /RGB_RED
- R11 pad 2: /CH14 -> Net-(LD2-Pad4)
- R12 pad 1: Net-(J1-Pad15) -> +3V3
- R12 pad 2: /CH15 -> /PGOOD_21V
- R13 pad 1: /ISET_1 -> +3V3
- R13 pad 2: GND -> /PGOOD_12V
- R14 pad 1: /ISET -> /VIN_CLEAN
- R14 pad 2: GND -> /PGOOD_5V
- R15 pad 1: /RGB_BLUE -> /VIN_CLEAN
- R15 pad 2: Net-(LD1-Pad6) -> Net-(R15-Pad2)
- R16 pad 1: /RGB_GREEN -> VDD
- R16 pad 2: Net-(LD1-Pad5) -> Net-(C4-Pad2)
- R17 pad 1: /RGB_RED -> Net-(C4-Pad2)
- R17 pad 2: Net-(LD1-Pad4) -> GND
- R18 pad 1: +3V3 -> Net-(R18-Pad1)
- R18 pad 2: /PGOOD_21V -> GND
- R19 pad 1: +3V3 -> +12V
- R19 pad 2: /PGOOD_12V -> Net-(C8-Pad2)
- R2 pad 2: /CH1 -> /ADC/CH1
- R20 pad 1: /VIN_CLEAN -> Net-(C8-Pad2)
- R20 pad 2: /Power Supplies/PG_5V -> GND
- R22 pad 1: VDD -> +5V
- R22 pad 2: Net-(C3-Pad2) -> Net-(C16-Pad2)
- R23 pad 1: Net-(C3-Pad2) -> Net-(R21-Pad2)
- R25 pad 1: +12V -> Net-(C16-Pad2)
- R25 pad 2: Net-(C7-Pad2) -> GND
- R26 pad 1: Net-(C7-Pad2) -> +3V3
- R26 pad 2: GND -> /~FAULT_SWITCH
- R27 pad 1: /VIN_CLEAN -> +3V3
- R27 pad 2: Net-(R27-Pad2) -> /PGOOD_SWITCH
- R28 pad 1: +5V -> +3V3
- R28 pad 2: Net-(C15-Pad2) -> /~EN_SWITCH
- R29 pad 1: Net-(R27-Pad2) -> +3V3
- R29 pad 2: GND -> /~FAULT_POE
- R3 pad 2: /CH2 -> /ADC/CH2
- R30 pad 1: Net-(R30-Pad1) -> +3V3
- R30 pad 2: GND -> /PGOOD_POE
- R31 pad 1: Net-(C15-Pad2) -> +3V3
- R31 pad 2: GND -> /~EN_POE
- R32 pad 1: +3V3 -> GND
- R32 pad 2: VDDA -> GNDA
- R33 pad 1: +3V3 -> Net-(C25-Pad1)
- R33 pad 2: /SCL -> Net-(C26-Pad1)
- R34 pad 1: +3V3 -> Net-(D1-Pad1)
- R34 pad 2: /SDA -> /ADC/VBAT
- R35 pad 1: GND -> Net-(C25-Pad1)
- R35 pad 2: GNDA -> /SCL
- R36 pad 1: +3V3 -> Net-(C25-Pad1)
- R36 pad 2: /~FAULT_POE -> /SDA
- R37 pad 1: +3V3 -> Net-(C25-Pad1)
- R37 pad 2: /PGOOD_POE -> Net-(R37-Pad2)
- R38 pad 1: +3V3 -> Net-(D1-Pad1)
- R38 pad 2: /~EN_POE -> GNDD
- R39 pad 2: /~FAULT_SWITCH -> /ADC/VDDA
- R4 pad 2: /CH3 -> /ADC/CH3
- R40 pad 2: /PGOOD_SWITCH -> /SCL
- R41 pad 2: /~EN_SWITCH -> /SDA
- R5 pad 1: Net-(J1-Pad1) -> /Network Switch Load Switch/ISET
- R5 pad 2: /CH8 -> GND
- R6 pad 1: Net-(J1-Pad3) -> /PoE Load Switch/ISET
- R6 pad 2: /CH9 -> GND
- R7 pad 1: Net-(J1-Pad5) -> /RGB_RED
- R7 pad 2: /CH10 -> Net-(LD1-Pad2)
- R8 pad 1: Net-(J1-Pad7) -> +3V3
- R8 pad 2: /CH11 -> Net-(LD1-Pad4)
- R9 pad 1: Net-(J1-Pad9) -> /RGB_BLUE
- R9 pad 2: /CH12 -> Net-(LD2-Pad6)
- RN1 pad 1: /CH15 -> GND
- RN1 pad 2: /CH14 -> GND
- RN1 pad 3: /CH13 -> GND
- RN1 pad 4: /CH12 -> GND
- RN1 pad 5: /CH11 -> /ADC/CH0
- RN1 pad 6: /CH10 -> /ADC/CH1
- RN1 pad 7: /CH9 -> /ADC/CH2
- RN1 pad 8: /CH8 -> /ADC/CH3
- U1 pad 12: Net-(C3-Pad2) -> Net-(C4-Pad2)
- U1 pad 13: Net-(C5-Pad1) -> Net-(C6-Pad1)
- U1 pad 14: Net-(C6-Pad1) -> Net-(C7-Pad1)
- U1 pad 15: Net-(C7-Pad2) -> Net-(C8-Pad2)
- U1 pad 17: Net-(R24-Pad1) -> Net-(R18-Pad1)
- U1 pad 18: /Power Supplies/PG_5V -> /PGOOD_5V
- U1 pad 5: Net-(R21-Pad2) -> Net-(R15-Pad2)
- U2 pad 1: /Power Supplies/PG_5V -> /PGOOD_5V
- U2 pad 10: Net-(C10-Pad2) -> Net-(C11-Pad2)
- U2 pad 14: Net-(R27-Pad2) -> Net-(R21-Pad2)
- U2 pad 17: Net-(R30-Pad1) -> Net-(R24-Pad1)
- U2 pad 18: Net-(C19-Pad1) -> Net-(C20-Pad1)
- U2 pad 19: Net-(C15-Pad2) -> Net-(C16-Pad2)
- U2 pad 20: Net-(C15-Pad2) -> Net-(C16-Pad2)
- U2 pad 3: Net-(C18-Pad1) -> Net-(C19-Pad1)
- U2 pad 7: Net-(C10-Pad1) -> Net-(C11-Pad1)
- U2 pad 8: Net-(C10-Pad2) -> Net-(C11-Pad2)
- U2 pad 9: Net-(C10-Pad2) -> Net-(C11-Pad2)
- U3 pad 1: (no net) -> +12V
- U3 pad 2: +5V -> /PGOOD_SWITCH
- U3 pad 3: no_connect_111 -> /Network Switch Load Switch/ISET
- U3 pad 4: GND -> /~EN_SWITCH
- U3 pad 5: no_connect_112 -> GND
- U3 pad 6: VDDA -> (no net)
- U3 pad 7: (no net) -> /~FAULT_SWITCH
- U3 pad 8: (no net) -> /Network Switch Load Switch/VOUT
- U4 pad 1: /SDA -> VDD
- U4 pad 2: /SCL -> /PGOOD_POE
- U4 pad 3: no_connect_113 -> /PoE Load Switch/ISET
- U4 pad 4: GND -> /~EN_POE
- U4 pad 6: GND -> (no net)
- U4 pad 7: GND -> /~FAULT_POE
- U4 pad 8: VDDA -> /PoE Injector/VDD_AP
- U5 pad 2: /SCL -> GND
- U5 pad 3: /SDA -> GND
- U5 pad 4: GND -> /PoE Injector/VDD_AP
- U5 pad 5: (no net) -> /PoE Injector/VDD_AP
- U5 pad 6: GND -> /PoE Injector/VDD_AP
- U6 pad 1: VDD -> Net-(C25-Pad1)
- U6 pad 2: /PGOOD_POE -> /ADC/VBAT
- U6 pad 3: /ISET -> GNDD
- U7 pad 1: +12V -> Net-(C26-Pad1)
- U7 pad 2: /PGOOD_SWITCH -> GNDD
- U7 pad 3: /ISET_1 -> (no net)
- U8 pad 1: GND -> Net-(R37-Pad2)
- U8 pad 2: GND -> no_connect_(U8-Pad2)
- U8 pad 3: GND -> /SCL
- U8 pad 4: /VOUT -> /SDA
- U8 pad 5: /VOUT -> GNDD
- U8 pad 6: /VOUT -> GNDD
- U8 pad 7: GND -> no_connect_(U8-Pad7)
Other:
- board size 100 x 130 mm -> 160 x 160 mm
- board text added: "Case is Hammond 1455R1602"
