File: vfc_power_supply.kicad_pcb (KiCad board)
At the start: 2 copper layers, 160 x 160 mm, 113 parts, among them J1 Conn_01x03_Male, J2 Conn_01x03_Male, J3 Conn_01x02_Male, J4 Raspberry_Pi_4B, J5 Connector_RJ45_Magjack_Abraco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, J6 Connector_RJ45_Magjack_Abraco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, M1 Logo_10mmx10mm, U1 LT8653S, U10 LM4040DBZ-3, U11 PCT2075D, U12 ADS7924, U2 LT8636, U3 FPF2701MPX, U4 FPF2701MPX, U5 TVS3300DRV, U6 LM3480-3.3, U7 LM4040DBZ-3, U8 ADS7924, U9 ISO1540

Commit message: Mostly complete, just missing a few tracks and review
Parts:
- removed the FL1 at (-54.5, 91.2)
- removed the R29 at (-58.0, 171.9)
- removed the R30 at (-53.2, 167.3)
- removed the R31 at (-58.0, 173.9)
- removed the R32 at (-42.7, 140.7)
- removed the R38 at (-23.8, 100.4)
- removed the U5 at (-43.1, 143.9)
- added C24: 47u, Capacitor_SMD:C_1206_3216Metric, F.Cu at (123.8, 167.8)
- added C25: 100n, Capacitor_SMD:C_0603_1608Metric, B.Cu at (151.6, 164.6)
- added C26: 100n, Capacitor_SMD:C_0603_1608Metric, B.Cu at (160.2, 163.6)
- added C27: 100n, Capacitor_SMD:C_0603_1608Metric, B.Cu at (158.2, 151.6)
- added C28: 100n, Capacitor_SMD:C_0603_1608Metric, B.Cu at (152.8, 151.5)
- added D1: P6SMB36CA-Q, Diode_SMD:D_SMB, B.Cu at (166.0, 158.2)
- added D3: 3V3, Diode_SMD:D_SOD-523, F.Cu at (34.5, 123.2)
- added D4: 3V3, Diode_SMD:D_SOD-523, F.Cu at (34.5, 119.8)
- added D5: 3V3, Diode_SMD:D_SOD-523, F.Cu at (31.0, 114.5)
- added FL2: EMI_Filter_CommonMode, Inductor_WUT:TDK_ACM7060-301-2PL-TL01, F.Cu at (34.8, 128.5)
- added J7: Conn_01x06_Female, Connector_WUT:Weidmuller_SL3.5-6-90G, F.Cu at (26.8, 125.0)
- added J8: Conn_01x06_Female, Connector_WUT:Weidmuller_SL3.5-6-90G, F.Cu at (26.8, 35.0)
- added J9: Conn_01x06_Female, Connector_WUT:Weidmuller_SL3.5-6-90G, F.Cu at (26.8, 65.0)
- added R11: 560k, Resistor_SMD:R_0603_1608Metric, F.Cu at (118.8, 161.0)
- added R34: 10K, Resistor_SMD:R_0603_1608Metric, F.Cu at (117.0, 169.0)
- added R35: 10K, Resistor_SMD:R_0603_1608Metric, F.Cu at (121.5, 161.0)
- added R36: 10K, Resistor_SMD:R_0603_1608Metric, F.Cu at (121.5, 157.0)
- added R37: DNF, Resistor_SMD:R_0603_1608Metric, B.Cu at (170.0, 170.0)
- added R43: 100k, Resistor_SMD:R_0603_1608Metric, F.Cu at (31.0, 123.2)
- added R44: 100k, Resistor_SMD:R_0603_1608Metric, F.Cu at (31.0, 119.8)
- added R45: 100k, Resistor_SMD:R_0603_1608Metric, F.Cu at (31.0, 116.2)
- added R5: 100, Resistor_SMD:R_0603_1608Metric, F.Cu at (32.5, 86.2)
- added R51: 1k, Resistor_SMD:R_0603_1608Metric, F.Cu at (48.5, 29.2)
- added R52: 1k, Resistor_SMD:R_0603_1608Metric, F.Cu at (48.5, 36.2)
- added R53: 1k, Resistor_SMD:R_0603_1608Metric, F.Cu at (48.5, 43.2)
- added R54: 1k, Resistor_SMD:R_0603_1608Metric, F.Cu at (30.2, 56.2)
- added R55: 1k, Resistor_SMD:R_0603_1608Metric, F.Cu at (30.2, 63.2)
- added R56: 1k, Resistor_SMD:R_0603_1608Metric, F.Cu at (30.2, 70.2)
- added R57: 10K, Resistor_SMD:R_0603_1608Metric, F.Cu at (48.5, 56.8)
- added R58: 10K, Resistor_SMD:R_0603_1608Metric, F.Cu at (48.5, 63.8)
- added R59: 10K, Resistor_SMD:R_0603_1608Metric, F.Cu at (48.5, 70.8)
- added R7: 100, Resistor_SMD:R_0603_1608Metric, F.Cu at (32.5, 93.2)
- added R8: 100, Resistor_SMD:R_0603_1608Metric, F.Cu at (32.5, 96.8)
- added R9: 100, Resistor_SMD:R_0603_1608Metric, F.Cu at (32.5, 100.2)
- added RN1: 10K, Resistor_SMD:R_Cat16-4, F.Cu at (36.2, 115.8)
- added U12: VO615A, Package_DIP:DIP-4_W8.89mm_SMDSocket_LongPads, F.Cu at (39.0, 28.0)
- added U13: VO615A, Package_DIP:DIP-4_W8.89mm_SMDSocket_LongPads, F.Cu at (39.0, 35.0)
- added U14: VO615A, Package_DIP:DIP-4_W8.89mm_SMDSocket_LongPads, F.Cu at (39.0, 42.0)
- added U15: VO615A, Package_DIP:DIP-4_W8.89mm_SMDSocket_LongPads, F.Cu at (39.0, 58.0)
- added U16: VO615A, Package_DIP:DIP-4_W8.89mm_SMDSocket_LongPads, F.Cu at (39.0, 65.0)
- added U17: VO615A, Package_DIP:DIP-4_W8.89mm_SMDSocket_LongPads, F.Cu at (39.2, 72.0)
- C11, C14, C15, C16, C19, C20, C21, C22, C23, C3: footprint Capacitor_SMD:C_0402_1005Metric -> Capacitor_SMD:C_0603_1608Metric
- C29: renamed from C24; footprint Capacitor_SMD:C_0402_1005Metric -> Capacitor_SMD:C_0603_1608Metric
- C30: renamed from C25; footprint Capacitor_SMD:C_0402_1005Metric -> Capacitor_SMD:C_0603_1608Metric
- C31: renamed from C26; footprint Capacitor_SMD:C_0402_1005Metric -> Capacitor_SMD:C_0603_1608Metric
- C32: renamed from C27; footprint Capacitor_SMD:C_0402_1005Metric -> Capacitor_SMD:C_0603_1608Metric
- C33: renamed from C28; footprint Capacitor_SMD:C_0402_1005Metric -> Capacitor_SMD:C_0603_1608Metric
- C34: renamed from C29; footprint Capacitor_SMD:C_0402_1005Metric -> Capacitor_SMD:C_0603_1608Metric
- C35: renamed from C30; footprint Capacitor_SMD:C_0402_1005Metric -> Capacitor_SMD:C_0603_1608Metric
- C36: renamed from C31; footprint Capacitor_SMD:C_0402_1005Metric -> Capacitor_SMD:C_0603_1608Metric
- C37: renamed from C32; footprint Capacitor_SMD:C_0402_1005Metric -> Capacitor_SMD:C_0603_1608Metric
- C38: renamed from C33; footprint Capacitor_SMD:C_0402_1005Metric -> Capacitor_SMD:C_0603_1608Metric
- C39: renamed from C34; footprint Capacitor_SMD:C_0402_1005Metric -> Capacitor_SMD:C_0603_1608Metric
- C4: renamed from C8; footprint Capacitor_SMD:C_0402_1005Metric -> Capacitor_SMD:C_0603_1608Metric
- C7: renamed from C6; footprint Capacitor_SMD:C_0402_1005Metric -> Capacitor_SMD:C_0603_1608Metric; moved to B.Cu
- C8: renamed from C7; footprint Capacitor_SMD:C_0402_1005Metric -> Capacitor_SMD:C_0603_1608Metric; moved to B.Cu
- C9: renamed from C4; footprint Capacitor_SMD:C_0402_1005Metric -> Capacitor_SMD:C_0603_1608Metric
- J2: value Conn_01x03_Male -> Conn_01x06_Female; footprint Connector_WUT:Powerpole_PP30-with-1377G2-PCB-pins-25A_3WAY -> Connector_WUT:Weidmuller_SL3.5-6-90G
- J5: value Connector_RJ45_Magjack_Abracon_ARJM11D7-502-AB-EW2 -> Connector_RJ45_Magjack_Abracon_ARJM11D7-502-NN-EW2; footprint Connector_WUT:Connector_RJ45_Magjack_Abracon_ARJM11D7-502-AB-EW2 -> Connector_WUT:Connector_RJ45_Magjack_Abracon_ARJM11D7-502-NN-EW2
- R1, R2: footprint Resistor_SMD:R_0402_1005Metric -> Resistor_SMD:R_0603_1608Metric
- R10: renamed from R5; footprint Resistor_SMD:R_0402_1005Metric -> Resistor_SMD:R_0603_1608Metric
- R12: renamed from R7; footprint Resistor_SMD:R_0402_1005Metric -> Resistor_SMD:R_0603_1608Metric
- R13: renamed from R8; footprint Resistor_SMD:R_0402_1005Metric -> Resistor_SMD:R_0603_1608Metric
- R14: renamed from R9; footprint Resistor_SMD:R_0402_1005Metric -> Resistor_SMD:R_0603_1608Metric
- R15: renamed from R10; footprint Resistor_SMD:R_0402_1005Metric -> Resistor_SMD:R_0603_1608Metric
- R16: renamed from R11; footprint Resistor_SMD:R_0402_1005Metric -> Resistor_SMD:R_0603_1608Metric
- R17: renamed from R12; footprint Resistor_SMD:R_0402_1005Metric -> Resistor_SMD:R_0603_1608Metric
- R18: renamed from R13; footprint Resistor_SMD:R_0402_1005Metric -> Resistor_SMD:R_0603_1608Metric
- R19: renamed from R14; footprint Resistor_SMD:R_0402_1005Metric -> Resistor_SMD:R_0603_1608Metric
- R20: renamed from R15; footprint Resistor_SMD:R_0402_1005Metric -> Resistor_SMD:R_0603_1608Metric
- R21: renamed from R19; footprint Resistor_SMD:R_0402_1005Metric -> Resistor_SMD:R_0603_1608Metric
- R22: renamed from R20; footprint Resistor_SMD:R_0402_1005Metric -> Resistor_SMD:R_0603_1608Metric
- R23: renamed from R18; footprint Resistor_SMD:R_0402_1005Metric -> Resistor_SMD:R_0603_1608Metric
- R24: renamed from R16; footprint Resistor_SMD:R_0402_1005Metric -> Resistor_SMD:R_0603_1608Metric
- R25: renamed from R17; footprint Resistor_SMD:R_0402_1005Metric -> Resistor_SMD:R_0603_1608Metric
- R26: renamed from R21; footprint Resistor_SMD:R_0402_1005Metric -> Resistor_SMD:R_0603_1608Metric
- R27: renamed from R22; footprint Resistor_SMD:R_0402_1005Metric -> Resistor_SMD:R_0603_1608Metric
- R28: renamed from R23; footprint Resistor_SMD:R_0402_1005Metric -> Resistor_SMD:R_0603_1608Metric
- R29: renamed from R24; footprint Resistor_SMD:R_0402_1005Metric -> Resistor_SMD:R_0603_1608Metric
- R3: renamed from R4; footprint Resistor_SMD:R_0402_1005Metric -> Resistor_SMD:R_0603_1608Metric
- R30: renamed from R25; footprint Resistor_SMD:R_0402_1005Metric -> Resistor_SMD:R_0603_1608Metric
- R31: renamed from R26; footprint Resistor_SMD:R_0402_1005Metric -> Resistor_SMD:R_0603_1608Metric
- R32: renamed from R27; footprint Resistor_SMD:R_0402_1005Metric -> Resistor_SMD:R_0603_1608Metric
- R33: renamed from R28; footprint Resistor_SMD:R_0402_1005Metric -> Resistor_SMD:R_0603_1608Metric
- R38: renamed from R33; footprint Resistor_SMD:R_0402_1005Metric -> Resistor_SMD:R_0603_1608Metric
- R39: renamed from R34; footprint Resistor_SMD:R_0402_1005Metric -> Resistor_SMD:R_0603_1608Metric
- R4: renamed from R3; footprint Resistor_SMD:R_0402_1005Metric -> Resistor_SMD:R_0603_1608Metric
- R40: renamed from R35; footprint Resistor_SMD:R_0402_1005Metric -> Resistor_SMD:R_0603_1608Metric
- R41: renamed from R36; footprint Resistor_SMD:R_0402_1005Metric -> Resistor_SMD:R_0603_1608Metric
- R42: renamed from R37; footprint Resistor_SMD:R_0402_1005Metric -> Resistor_SMD:R_0603_1608Metric
- R46: renamed from R39; footprint Resistor_SMD:R_0402_1005Metric -> Resistor_SMD:R_0603_1608Metric
- R47: renamed from R40; footprint Resistor_SMD:R_0402_1005Metric -> Resistor_SMD:R_0603_1608Metric
- R48: renamed from R41; footprint Resistor_SMD:R_0402_1005Metric -> Resistor_SMD:R_0603_1608Metric
- R49: renamed from R42; footprint Resistor_SMD:R_0402_1005Metric -> Resistor_SMD:R_0603_1608Metric
- R50: renamed from R43; footprint Resistor_SMD:R_0402_1005Metric -> Resistor_SMD:R_0603_1608Metric
- R6: value 560k -> 100; footprint Resistor_SMD:R_0402_1005Metric -> Resistor_SMD:R_0603_1608Metric
- moved M1 249.1 mm to (115.2, 25.0)
- moved C13 248.3 mm to (129.8, 41.2), turned to 90 degrees
- moved C12 246.3 mm to (142.8, 41.2), turned to 90 degrees
- moved L3 242.1 mm to (136.2, 42.8), turned to 180 degrees
- moved R13 226.8 mm to (168.0, 54.8)
- moved R12 218.3 mm to (168.0, 57.2)
- moved C23 198.2 mm to (159.0, 134.0), turned to 180 degrees
- moved R15 193.0 mm to (93.8, 104.5), turned to 180 degrees
- moved R14 192.9 mm to (93.8, 102.8), turned to 180 degrees
- moved R3 192.5 mm to (109.0, 134.8)
- moved L4 189.4 mm to (100.8, 128.8)
- moved R16 179.8 mm to (93.8, 106.2), turned to 180 degrees
- moved U4 176.2 mm to (119.2, 165.5), turned to -90 degrees
- moved C10 176.1 mm to (91.8, 148.8), turned to 90 degrees
- moved R2 175.5 mm to (91.5, 141.3)
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- renumbered C5 to C10, C9 to C5, C10 to C6, D1 to D2, D2 to D6, D3 to D7, D4 to D8, D5 to D9, FL2 to FL1, L2 to L1, L1 to L2, RN1 to RN2, TP2 to TP1, TP1 to TP2, U11 to U10, U12 to U11, U6 to U5, U7 to U6, U8 to U7, U9 to U8, U10 to U9
Connections:
- net no_connect_(U11-Pad3) renamed no_connect_(U10-Pad3)
- net no_connect_(U11-Pad5) renamed no_connect_(U10-Pad5)
- net no_connect_(U12-Pad2) renamed no_connect_(U11-Pad2)
- net no_connect_(U8-Pad2) renamed no_connect_(U7-Pad2)
- net no_connect_(U8-Pad7) renamed no_connect_(U7-Pad7)
- C4 pad 2: Net-(C8-Pad2) -> Net-(C4-Pad2)
- C9 pad 2: Net-(C4-Pad2) -> Net-(C9-Pad2)
- FL1 pad 1: /Network Switch Load Switch/VOUT -> Net-(C1-Pad1)
- FL1 pad 2: Net-(C1-Pad1) -> /Network Switch Load Switch/VOUT
- FL1 pad 3: GND -> Net-(C1-Pad2)
- FL1 pad 4: Net-(C1-Pad2) -> GND
- J2 pad 2: no_connect_(J2-Pad2) -> Net-(J2-Pad2)
- J4 pad 10: no_connect_(J4-Pad10) -> /GPIO15/RXD
- J4 pad 11: /RGB_BLUE -> /RGB_RED
- J4 pad 15: /RGB_RED -> /RGB_BLUE
- J4 pad 19: no_connect_(J4-Pad19) -> /GPIO10/SDA
- J4 pad 21: no_connect_(J4-Pad21) -> /GPIO9/SCL
- J4 pad 22: no_connect_(J4-Pad22) -> /PGOOD_5V
- J4 pad 23: /PGOOD_SWITCH -> /OPTO_IN_2
- J4 pad 24: no_connect_(J4-Pad24) -> /~FAULT_SWITCH
- J4 pad 29: /~FAULT_SWITCH -> /OPTO_IN_1
- J4 pad 31: /PGOOD_POE -> /OPTO_IN_0
- J4 pad 32: no_connect_(J4-Pad32) -> /PGOOD_SWITCH
- J4 pad 33: /~EN_POE -> /OPTO_OUT_2
- J4 pad 35: /~FAULT_POE -> /OPTO_OUT_1
- J4 pad 36: no_connect_(J4-Pad36) -> /~FAULT_POE
- J4 pad 37: no_connect_(J4-Pad37) -> /OPTO_OUT_0
- J4 pad 38: no_connect_(J4-Pad38) -> /~EN_POE
- J4 pad 40: no_connect_(J4-Pad40) -> /PGOOD_POE
- J4 pad 7: no_connect_(J4-Pad7) -> /GPIO4/ONE_WIRE
- J4 pad 8: /PGOOD_5V -> /GPIO14/TXD
- J6 pad 1: no_connect_(J6-Pad1) -> Net-(C27-Pad1)
- J6 pad 12: no_connect_(J6-Pad12) -> Net-(C25-Pad1)
- J6 pad 6: no_connect_(J6-Pad6) -> Net-(C26-Pad1)
- J6 pad 7: no_connect_(J6-Pad7) -> Net-(C28-Pad1)
- L1 pad 1: Net-(L2-Pad1) -> Net-(L1-Pad1)
- L2 pad 1: Net-(L1-Pad1) -> Net-(L2-Pad1)
- R1 pad 2: /ADC/CH0 -> /ADC/CH1
- R17 pad 2: /PGOOD_21V -> /PGOOD_12V
- R18 pad 2: /PGOOD_12V -> /PGOOD_21V
- R2 pad 2: /ADC/CH1 -> /ADC/CH0
- R21 pad 2: Net-(C8-Pad2) -> Net-(C4-Pad2)
- R22 pad 1: Net-(C8-Pad2) -> Net-(C4-Pad2)
- R24 pad 2: Net-(C4-Pad2) -> Net-(C9-Pad2)
- R25 pad 1: Net-(C4-Pad2) -> Net-(C9-Pad2)
- R3 pad 2: /ADC/CH3 -> /ADC/CH2
- R30 pad 1: Net-(C16-Pad2) -> GND
- R30 pad 2: GND -> Net-(C16-Pad2)
- R4 pad 2: /ADC/CH2 -> /ADC/CH3
- R40 pad 2: /SCL -> Net-(R40-Pad2)
- R41 pad 2: /SDA -> Net-(R41-Pad2)
- R6 pad 1: /PoE Load Switch/ISET -> /GPIO10/SDA
- R6 pad 2: GND -> Net-(J2-Pad2)
- U1 pad 15: Net-(C8-Pad2) -> Net-(C9-Pad2)
- U1 pad 3: /PGOOD_12V -> /PGOOD_21V
- U1 pad 4: /PGOOD_21V -> /PGOOD_12V
- U10 pad 7: no_connect_(U11-Pad7) -> no_connect_(U10-Pad7)
- U11 pad 7: no_connect_(U12-Pad7) -> no_connect_(U11-Pad7)
- U7 pad 10: no_connect_(U8-Pad10) -> Net-(D4-Pad1)
- U7 pad 11: no_connect_(U8-Pad11) -> Net-(D3-Pad1)
- U7 pad 3: /SCL -> Net-(R40-Pad2)
- U7 pad 4: /SDA -> Net-(R41-Pad2)
- U7 pad 9: no_connect_(U8-Pad9) -> Net-(D5-Pad1)
- U8 pad 6: /SCL -> Net-(R40-Pad2)
- U8 pad 7: /SDA -> Net-(R41-Pad2)
Routing:
- net /OPTO_OUT_0: track 0.00 -> 151.1 mm
- net /OPTO_OUT_1: track 0.00 -> 144.6 mm
- net /OPTO_OUT_2: track 0.00 -> 140.6 mm
- net /OPTO_IN_0: track 0.00 -> 138.9 mm
- net /OPTO_IN_1: track 0.00 -> 130.5 mm
- net /~EN_SWITCH: track 0.00 -> 120.8 mm
- net /~FAULT_SWITCH: track 0.00 -> 118.8 mm
- net /RGB_RED: track 0.00 -> 117.3 mm, vias 0 -> 1
- net /OPTO_IN_2: track 0.00 -> 116.8 mm
- net /GPIO9/SCL: track 0.00 -> 116.5 mm
- net /PGOOD_SWITCH: track 0.00 -> 116.3 mm
- net /GPIO10/SDA: track 0.00 -> 111.1 mm
- net /GPIO15/RXD: track 0.00 -> 100.4 mm, vias 0 -> 1
- net /GPIO14/TXD: track 0.00 -> 96.4 mm, vias 0 -> 1
- net /GPIO4/ONE_WIRE: track 0.00 -> 90.2 mm, vias 0 -> 1
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- added copper zone on F.Cu, net +12V
- added copper zone on In2.Cu, net +12V
- added copper zone on In2.Cu, net +3V3
- added copper zone on F.Cu, net +5V
- added copper zone on B.Cu, net /VIN_CLEAN
- added copper zone on F.Cu, net /VIN_CLEAN
- added copper zone on F.Cu, net GND
- added copper zone on In1.Cu, net GND
- added copper zone on B.Cu, net GNDA
- added copper zone on F.Cu, net GNDD
- added copper zone on In1.Cu, net GNDD
- added copper zone on F.Cu, net Net-(C11-Pad2)
- added copper zone on F.Cu, net Net-(L1-Pad1)
- added copper zone on F.Cu, net Net-(L2-Pad1)
- added copper zone on F.Cu, net VDD
- added copper zone on In2.Cu, net VDD
Other:
- outline, holes or cut-outs redrawn
- copper layers 2 -> 4
